File: NIVARA_PCB/NIVARA/NIVARA.kicad_pcb (KiCad board)
At the start: 2 copper layers, 0 parts

Commit message: ACTUALIZACION
Parts:
- added C1: 10uF, PCM_Capacitor_SMD_AKL:C_0603_1608Metric, F.Cu at (-76.4, 98.8)
- added C10: C_0603, PCM_Capacitor_SMD_AKL:C_0603_1608Metric, F.Cu at (-12.1, 78.2)
- added C11: C_0603, PCM_Capacitor_SMD_AKL:C_0603_1608Metric, F.Cu at (-12.1, 80.9)
- added C12: C_0603, PCM_Capacitor_SMD_AKL:C_0603_1608Metric, F.Cu at (-12.1, 95.5)
- added C13: C_0603, PCM_Capacitor_SMD_AKL:C_0603_1608Metric, F.Cu at (-12.1, 98.2)
- added C2: 100nF, PCM_Capacitor_SMD_AKL:C_0603_1608Metric, F.Cu at (-76.4, 101.5)
- added C3: C_0603, PCM_Capacitor_SMD_AKL:C_0603_1608Metric, F.Cu at (-76.4, 104.2)
- added C4: 22uF, PCM_Capacitor_SMD_AKL:C_0603_1608Metric, F.Cu at (-76.4, 106.9)
- added C5: 22uF, PCM_Capacitor_SMD_AKL:C_0603_1608Metric, F.Cu at (-76.4, 109.6)
- added D1: 1N4007, Diode_SMD:D_SOD-123F, F.Cu at (-49.1, 49.3)
- added D2: 1N4007, Diode_SMD:D_SOD-123F, F.Cu at (-49.1, 66.3)
- added D3: SMBJ12CA, PCM_Diode_SMD_AKL:D_SMB_TVS, F.Cu at (-44.1, 95.6)
- added H1: MountingHole_Pad, MountingHole:MountingHole_2.2mm_M2_Pad_Via, F.Cu at (154.9, 76.0)
- added H2: MountingHole_Pad, MountingHole:MountingHole_2.2mm_M2_Pad_Via, F.Cu at (69.9, 126.0)
- added J1: Screw_Terminal_01x02, TerminalBlock:TerminalBlock_bornier-2_P5.08mm, F.Cu at (71.1, 138.2)
- added J2: Screw_Terminal_01x02, TerminalBlock:TerminalBlock_bornier-2_P5.08mm, F.Cu at (-75.3, 54.7)
- added J3: I_NPN, TerminalBlock:TerminalBlock_bornier-2_P5.08mm, F.Cu at (-75.3, 63.7)
- added J4: I_PNP, TerminalBlock:TerminalBlock_bornier-2_P5.08mm, F.Cu at (-75.3, 72.8)
- added J5: RELAY_1, TerminalBlock:TerminalBlock_bornier-3_P5.08mm, F.Cu at (-84.1, 35.2)
- added J6: RELAY_2, TerminalBlock:TerminalBlock_bornier-3_P5.08mm, F.Cu at (-84.0, 44.7)
- added J7: O_NPN, TerminalBlock:TerminalBlock_bornier-2_P5.08mm, F.Cu at (-75.3, 81.8)
- added J8: O_PNP, TerminalBlock:TerminalBlock_bornier-2_P5.08mm, F.Cu at (-75.3, 90.9)
- added JP1: SolderJumper_2_Open, Jumper:SolderJumper-2_P1.3mm_Open_RoundedPad1.0x1.5mm, F.Cu at (-67.9, 99.2)
- added L1: L_Iron, Inductor_SMD:L_0201_0603Metric_Pad0.64x0.40mm_HandSolder, F.Cu at (-69.7, 108.3)
- added LED5: LED_0603_Green, PCM_LED_SMD_AKL:LED_0603_1608Metric, F.Cu at (-14.8, 87.0)
- added LED6: LED_0603_Green, PCM_LED_SMD_AKL:LED_0603_1608Metric, F.Cu at (-14.8, 90.3)
- added LED7: LED_0603_Green, PCM_LED_SMD_AKL:LED_0603_1608Metric, F.Cu at (-14.8, 104.3)
- added LED8: LED_0603_Green, PCM_LED_SMD_AKL:LED_0603_1608Metric, F.Cu at (-14.8, 107.6)
- added Q1: PMBT3904, PCM_Package_TO_SOT_SMD_AKL:SOT-23, F.Cu at (-49.6, 53.6)
- added Q2: PMBT3904, PCM_Package_TO_SOT_SMD_AKL:SOT-23, F.Cu at (-49.8, 70.8)
- added R1: 22K, PCM_Resistor_SMD_AKL:R_0603_1608Metric, F.Cu at (-72.1, 98.8)
- added R19: 10K, PCM_Resistor_SMD_AKL:R_0603_1608Metric, F.Cu at (-25.0, 78.2)
- added R2: 22K, PCM_Resistor_SMD_AKL:R_0603_1608Metric, F.Cu at (-72.1, 101.5)
- added R20: ?, PCM_Resistor_SMD_AKL:R_0603_1608Metric, F.Cu at (-25.0, 80.9)
- added R21: 1K, PCM_Resistor_SMD_AKL:R_1206_3216Metric_Pad1.30x1.75mm_HandSolder, F.Cu at (-19.9, 90.4)
- added R22: 10K, PCM_Resistor_SMD_AKL:R_0603_1608Metric, F.Cu at (-25.0, 83.6)
- added R23: ?, PCM_Resistor_SMD_AKL:R_0603_1608Metric, F.Cu at (-25.0, 86.3)
- added R24: 1K, PCM_Resistor_SMD_AKL:R_1206_3216Metric_Pad1.30x1.75mm_HandSolder, F.Cu at (-19.9, 104.3)
- added R25: 1K, PCM_Resistor_SMD_AKL:R_1206_3216Metric_Pad1.30x1.75mm_HandSolder, F.Cu at (-19.9, 107.7)
- added R26: 10K, PCM_Resistor_SMD_AKL:R_0603_1608Metric, F.Cu at (-25.0, 95.5)
- added R27: 10K, PCM_Resistor_SMD_AKL:R_0603_1608Metric, F.Cu at (-25.0, 98.2)
- added R28: ?, PCM_Resistor_SMD_AKL:R_0603_1608Metric, F.Cu at (-25.0, 100.9)
- added R29: ?, PCM_Resistor_SMD_AKL:R_0603_1608Metric, F.Cu at (-25.0, 103.6)
- added R30: 22K, PCM_Resistor_SMD_AKL:R_0603_1608Metric, F.Cu at (-25.8, 42.5)
- added R31: ?, PCM_Resistor_SMD_AKL:R_0603_1608Metric, F.Cu at (-25.8, 45.2)
- added R32: 22K, PCM_Resistor_SMD_AKL:R_0603_1608Metric, F.Cu at (-25.8, 47.9)
- added R33: ?, PCM_Resistor_SMD_AKL:R_0603_1608Metric, F.Cu at (-25.8, 50.6)
- added R34: 47K, PCM_Resistor_SMD_AKL:R_0603_1608Metric, F.Cu at (-37.8, 94.1)
- added R35: 47K, PCM_Resistor_SMD_AKL:R_0603_1608Metric, F.Cu at (-37.8, 96.8)
- added R4: 1K, PCM_Resistor_SMD_AKL:R_1206_3216Metric_Pad1.30x1.75mm_HandSolder, F.Cu at (-19.9, 87.0)
- added RLY1: SRD-24VDC-SL-C, easyeda2kicad:RELAY-TH_SRD-XXVDC-XL-C, F.Cu at (-39.0, 49.5)
- added RLY2: SRD-24VDC-SL-C, easyeda2kicad:RELAY-TH_SRD-XXVDC-XL-C, F.Cu at (-39.0, 66.4)
- added TP1: TestPoint, TestPoint:TestPoint_THTPad_D1.0mm_Drill0.5mm, F.Cu at (-72.7, 109.0)
- added TP6: TestPoint, TestPoint:TestPoint_THTPad_D1.0mm_Drill0.5mm, F.Cu at (-11.2, 86.8)
- added TP7: TestPoint, TestPoint:TestPoint_THTPad_D1.0mm_Drill0.5mm, F.Cu at (-11.2, 89.9)
- added TP8: TestPoint, TestPoint:TestPoint_THTPad_D1.0mm_Drill0.5mm, F.Cu at (-11.2, 104.1)
- added TP9: TestPoint, TestPoint:TestPoint_THTPad_D1.0mm_Drill0.5mm, F.Cu at (-11.2, 107.2)
- added U1: AP63203WU, Package_TO_SOT_SMD:TSOT-23-6, F.Cu at (-71.6, 105.2)
- added U2: AT3H4A-CUH-S, easyeda2kicad:SSOP-4_L2.7-W4.6-P1.27-LS7.0-TL, F.Cu at (-18.6, 79.1)
- added U4: AT3H4A-CUH-S, easyeda2kicad:SSOP-4_L2.7-W4.6-P1.27-LS7.0-TL, F.Cu at (-18.6, 83.3)
- added U5: AT3H4A-CUH-S, easyeda2kicad:SSOP-4_L2.7-W4.6-P1.27-LS7.0-TL, F.Cu at (-18.6, 96.4)
- added U6: AT3H4A-CUH-S, easyeda2kicad:SSOP-4_L2.7-W4.6-P1.27-LS7.0-TL, F.Cu at (-18.6, 100.6)
- added U7: TD321D485H-A-LB, TD321D485H-A-LB:TD321D485H-A-LB, F.Cu at (-38.7, 84.7)
Other:
- board outline added: 101.2 x 82 mm

Commit message: avance
Parts:
- removed J2: Screw_Terminal_01x02, TerminalBlock:TerminalBlock_bornier-2_P5.08mm
- added C14: C_0603, PCM_Capacitor_SMD_AKL:C_0603_1608Metric, F.Cu at (-56.9, -41.4)
- added C15: C_0603, PCM_Capacitor_SMD_AKL:C_0603_1608Metric, F.Cu at (-56.9, -38.6)
- added C6: 100nF, PCM_Capacitor_SMD_AKL:C_0603_1608Metric, F.Cu at (5.84, -5.13)
- added C7: 100nF, PCM_Capacitor_SMD_AKL:C_0603_1608Metric, F.Cu at (5.84, -0.41)
- added C8: 100nF, PCM_Capacitor_SMD_AKL:C_0603_1608Metric, F.Cu at (5.84, 4.31)
- added J10: I_ANALOG, TerminalBlock:TerminalBlock_bornier-4_P5.08mm, F.Cu at (138.6, 138.2)
- added J11: RS485, TerminalBlock:TerminalBlock_bornier-3_P5.08mm, F.Cu at (121.1, 138.2)
- added J12: O_ANALOG, TerminalBlock:TerminalBlock_bornier-4_P5.08mm, F.Cu at (153.1, 63.6)
- added J9: I_DIG, TerminalBlock:TerminalBlock_bornier-2_P5.08mm, F.Cu at (108.6, 138.2)
- added LED10: LED_0603_Green, PCM_LED_SMD_AKL:LED_0603_1608Metric, F.Cu at (-59.6, -29.2)
- added LED9: LED_0603_Green, PCM_LED_SMD_AKL:LED_0603_1608Metric, F.Cu at (-59.6, -32.6)
- added R3: 22K, PCM_Resistor_SMD_AKL:R_0603_1608Metric, F.Cu at (-42.3, -33.2)
- added R36: ?, PCM_Resistor_SMD_AKL:R_1206_3216Metric_Pad1.30x1.75mm_HandSolder, F.Cu at (-64.7, -29.1)
- added R37: 10K, PCM_Resistor_SMD_AKL:R_0603_1608Metric, F.Cu at (-69.8, -41.4)
- added R38: 10K, PCM_Resistor_SMD_AKL:R_0603_1608Metric, F.Cu at (-69.8, -38.6)
- added R39: ?, PCM_Resistor_SMD_AKL:R_0603_1608Metric, F.Cu at (-69.8, -35.9)
- added R40: ?, PCM_Resistor_SMD_AKL:R_0603_1608Metric, F.Cu at (-69.8, -33.2)
- added R41: 10K, PCM_Resistor_SMD_AKL:R_0603_1608Metric, F.Cu at (-42.3, -30.5)
- added R42: 10K, PCM_Resistor_SMD_AKL:R_0603_1608Metric, F.Cu at (-42.3, -38.0)
- added R5: ?, PCM_Resistor_SMD_AKL:R_1206_3216Metric_Pad1.30x1.75mm_HandSolder, F.Cu at (-64.7, -32.5)
- added R6: 1K, PCM_Resistor_SMD_AKL:R_1206_3216Metric_Pad1.30x1.75mm_HandSolder, F.Cu at (-41.3, -41.0)
- added TP10: TestPoint, TestPoint:TestPoint_THTPad_D1.0mm_Drill0.5mm, F.Cu at (-56.0, -32.7)
- added TP11: TestPoint, TestPoint:TestPoint_THTPad_D1.0mm_Drill0.5mm, F.Cu at (-56.0, -29.7)
- added U10: GP8201S-TC50-EW, easyeda2kicad:ESOP-8_L4.9-W3.9-P1.27-LS6.0-BL-EP, F.Cu at (-1.51, -2.48)
- added U3: AT3H4A-CUH-S, easyeda2kicad:SSOP-4_L2.7-W4.6-P1.27-LS7.0-TL, F.Cu at (-64.1, -40.6)
- added U8: AT3H4A-CUH-S, easyeda2kicad:SSOP-4_L2.7-W4.6-P1.27-LS7.0-TL, F.Cu at (-63.4, -36.2)
- added U9: GP8303-TC50-EW, easyeda2kicad:ESOP-10_L4.9-W3.9-P1.00-LS6.1-BL-EP, F.Cu at (-49.4, -38.7)
- J1: value Screw_Terminal_01x02 -> Power
- moved J6 215.4 mm to (130.6, 63.6), turned to 180 degrees
- moved J5 199.5 mm to (113.3, 63.6), turned to 180 degrees
- moved J4 183.7 mm to (96.3, 138.2)
- moved J3 175.6 mm to (83.7, 138.2)
- moved J8 173.5 mm to (96.0, 63.6), turned to 180 degrees
- moved U7 169.3 mm to (126.1, 123.5), turned to 180 degrees
- moved RLY1 167.3 mm to (125.6, 79.3), turned to 90 degrees
- moved J7 160.1 mm to (83.7, 63.6), turned to 180 degrees
- moved RLY2 147.8 mm to (108.2, 79.4), turned to 90 degrees
- moved U1 87.2 mm to (-158.8, 100.9)
- moved C1 87.2 mm to (-163.5, 94.5)
- moved C2 87.2 mm to (-163.5, 97.2)
- moved C3 87.2 mm to (-163.5, 99.9)
- moved C4 87.2 mm to (-163.5, 102.6)
- moved C5 87.2 mm to (-163.5, 105.3)
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Connections:
- net /NIVARA_BOARD/IN NPN/OUT_1 renamed /NIVARA_BOARD/ESP32 S3/NPN_IN1
- net /NIVARA_BOARD/IN NPN/OUT_2 renamed /NIVARA_BOARD/ESP32 S3/NPN_IN2
- net /NIVARA_BOARD/IN PNP/OUT_1 renamed /NIVARA_BOARD/ESP32 S3/PNP_IN1
- net /NIVARA_BOARD/IN PNP/OUT_2 renamed /NIVARA_BOARD/ESP32 S3/PNP_IN2
- net /NIVARA_BOARD/RS_485/RX renamed /NIVARA_BOARD/ESP32 S3/RX
- net /NIVARA_BOARD/RS_485/TX renamed /NIVARA_BOARD/ESP32 S3/TX
- J1 pad 1: GND -> VCC
- J1 pad 2: VCC -> GND
- J3 pad 1: /NIVARA_BOARD/NPN_IN2 -> /NIVARA_BOARD/PNP_IN1
- J3 pad 2: /NIVARA_BOARD/NPN_IN1 -> /NIVARA_BOARD/PNP_IN2
- J4 pad 1: /NIVARA_BOARD/PNP_IN2 -> /NIVARA_BOARD/NPN_IN1
- J4 pad 2: /NIVARA_BOARD/PNP_IN1 -> /NIVARA_BOARD/NPN_IN2
- J5 pad 1: /NIVARA_BOARD/REL_NC2 -> /NIVARA_BOARD/REL_NO2
- J5 pad 3: /NIVARA_BOARD/REL_NO2 -> /NIVARA_BOARD/REL_NC2
- J6 pad 1: /NIVARA_BOARD/REL_NC1 -> /NIVARA_BOARD/REL_NO1
- J6 pad 3: /NIVARA_BOARD/REL_NO1 -> /NIVARA_BOARD/REL_NC1
Routing:
- added copper zone on B.Cu, net GND
Other:
- copper layers 2 -> 4
