File: NIVARA_PCB/NIVARA/NIVARA.kicad_pcb (KiCad board)
At the start: 4 copper layers, 101.2 x 82 mm, 174 parts, among them IC1 ITS5215, J1 Power, J10 I_ANALOG, J11 RS485, J12 O_ANALOG, J3 I_NPN, J4 I_PNP, J5 RELAY_1, J6 RELAY_2, J7 O_NPN, J8 O_PNP, J9 I_DIG, Q1 DMP3056L, Q2 PMBT3904, Q4 PMBT3904, U1 AP63203WU, U10 GP8201S-TC50-EW, U11 ESP32-S3-WROOM-1, U12 ZMM12V_C5345999, U13 GP8201S-TC50-EW, U14 ZXMS6004FFQTA, U15 ZXMS6004FFQTA, U2 AT3H4A-CUH-S, U3 AT3H4A-CUH-S, U4 AT3H4A-CUH-S, U5 AT3H4A-CUH-S, U6 AT3H4A-CUH-S, U7 TD321D485H-A-LB, U8 AT3H4A-CUH-S, U9 GP8303-TC50-EW

Commit message: se extendio GND
Parts:
- added kibuzzard-68A4ACEC: G***, kibuzzard-68A4ACEC, F.Cu at (71.4, 69.4)
- added kibuzzard-68A4AD1D: G***, kibuzzard-68A4AD1D, F.Cu at (76.5, 69.4)
- added kibuzzard-68A4AD43: G***, kibuzzard-68A4AD43, F.Cu at (83.6, 69.4)
- added kibuzzard-68A4AD55: G***, kibuzzard-68A4AD55, F.Cu at (88.7, 69.4)
- added kibuzzard-68A4AE0E: G***, kibuzzard-68A4AE0E, F.Cu at (95.8, 69.4)
- added kibuzzard-68A4AE1F: G***, kibuzzard-68A4AE1F, F.Cu at (100.9, 69.4)
- added kibuzzard-68A4AE2A: G***, kibuzzard-68A4AE2A, F.Cu at (106.0, 69.4)
- added kibuzzard-68A4AE4D: G***, kibuzzard-68A4AE4D, F.Cu at (113.1, 69.4)
- added kibuzzard-68A4AE56: G***, kibuzzard-68A4AE56, F.Cu at (118.2, 69.4)
- added kibuzzard-68A4AE5E: G***, kibuzzard-68A4AE5E, F.Cu at (123.3, 69.4)
- added kibuzzard-68A4AF27: G***, kibuzzard-68A4AF27, F.Cu at (132.9, 69.4)
- added kibuzzard-68A4AF38: G***, kibuzzard-68A4AF38, F.Cu at (137.7, 69.4)
- added kibuzzard-68A4AF50: G***, kibuzzard-68A4AF50, F.Cu at (143.3, 69.4)
- added kibuzzard-68A4AF5B: G***, kibuzzard-68A4AF5B, F.Cu at (148.1, 69.4)
- added kibuzzard-68A4B644: G***, kibuzzard-68A4B644, F.Cu at (64.5, 135.4)
- added kibuzzard-68A4B67A: G***, kibuzzard-68A4B67A, F.Cu at (160.2, 65.9)
Routing:
- net +3V3: track 8.82 -> 100.3 mm
- net VCC: track 51.3 -> 76.3 mm, vias 23 -> 44
- net /NIVARA_BOARD/OUT A 4-20mA/A2: track 2.18 -> 16.3 mm
- net /NIVARA_BOARD/RS_A: track 7.91 -> 20.3 mm
- net Net-(LED8-A): track 0.00 -> 10.6 mm, vias 0 -> 2
- net /NIVARA_BOARD/PNP_OUT1: track 0.00 -> 9.96 mm
- net /NIVARA_BOARD/PNP_OUT2: track 0.00 -> 9.59 mm
- net Net-(Q1-G): track 0.00 -> 8.51 mm
- net /NIVARA_BOARD/RS_B: track 6.90 -> 15.0 mm
- net /NIVARA_BOARD/NPN_OUT2: track 0.00 -> 7.89 mm
- net /NIVARA_BOARD/NPN_OUT1: track 0.00 -> 7.89 mm
- net Net-(U9-SET): track 0.00 -> 7.16 mm
- net Net-(Q1-S): track 0.00 -> 5.03 mm
- net Net-(U15-IN): track 0.00 -> 4.14 mm
- net Net-(U14-IN): track 0.00 -> 4.05 mm
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