File: NIVARA_PCB/NIVARA/NIVARA.kicad_pcb (KiCad board)
At the start: 4 copper layers, 101.2 x 82 mm, 200 parts, among them IC1 ITS5215, J1 Power, J10 I_ANALOG, J11 RS485, J12 O_ANALOG, J3 I_NPN, J4 I_PNP, J5 RELAY_1, J6 RELAY_2, J7 O_NPN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

Commit message: RUTEO ENTRADAS
Connections:
- U11 pad 10: /NIVARA_BOARD/ESP32 S3/NPN_OUT2 -> /NIVARA_BOARD/ESP32 S3/NPN_OUT1
- U11 pad 11: /NIVARA_BOARD/ESP32 S3/NPN_OUT1 -> /NIVARA_BOARD/ESP32 S3/NPN_OUT2
- U11 pad 18: unconnected-(U11-GPIO10/TOUCH10/ADC1_CH9/FSPICS0/FSPIIO4/SUBSPICS0-Pad18) -> /NIVARA_BOARD/ESP32 S3/RX
- U11 pad 19: unconnected-(U11-GPIO11/TOUCH11/ADC2_CH0/FSPID/FSPIIO5/SUBSPID-Pad19) -> /NIVARA_BOARD/ESP32 S3/TX
- U11 pad 20: unconnected-(U11-GPIO12/TOUCH12/ADC2_CH1/FSPICLK/FSPIIO6/SUBSPICLK-Pad20) -> /NIVARA_BOARD/ESP32 S3/DRY_IN2
- U11 pad 21: unconnected-(U11-GPIO13/TOUCH13/ADC2_CH2/FSPIQ/FSPIIO7/SUBSPIQ-Pad21) -> /NIVARA_BOARD/ESP32 S3/DRY_IN1
- U11 pad 23: unconnected-(U11-GPIO21-Pad23) -> /NIVARA_BOARD/ESP32 S3/PNP_IN2
- U11 pad 24: unconnected-(U11-GPIO47/SPICLK_P/SUBSPICLK_P_DIFF-Pad24) -> /NIVARA_BOARD/ESP32 S3/PNP_IN1
- U11 pad 25: /NIVARA_BOARD/ESP32 S3/RX -> /NIVARA_BOARD/ESP32 S3/NPN_IN2
- U11 pad 26: /NIVARA_BOARD/ESP32 S3/TX -> /NIVARA_BOARD/ESP32 S3/NPN_IN1
Routing:
- net /NIVARA_BOARD/ESP32 S3/NPN_OUT2: track 0.00 -> 113.9 mm, vias 0 -> 2
- net /NIVARA_BOARD/ESP32 S3/NPN_OUT1: track 0.00 -> 111.3 mm, vias 0 -> 2
- net /NIVARA_BOARD/ESP32 S3/NPN_IN1: track 4.30 -> 70.5 mm, vias 0 -> 2
- net /NIVARA_BOARD/ESP32 S3/NPN_IN2: track 2.55 -> 61.9 mm, vias 0 -> 2
- net /NIVARA_BOARD/ESP32 S3/PNP_IN1: track 3.17 -> 55.0 mm, vias 0 -> 2
- net /NIVARA_BOARD/ESP32 S3/PNP_IN2: track 2.71 -> 47.5 mm, vias 0 -> 2
- net /NIVARA_BOARD/ESP32 S3/DRY_IN1: track 2.72 -> 40.6 mm, vias 0 -> 2
- net /NIVARA_BOARD/ESP32 S3/DRY_IN2: track 3.33 -> 35.2 mm, vias 0 -> 2
- net /NIVARA_BOARD/ESP32 S3/TX: track 0.00 -> 23.8 mm, vias 0 -> 1
- net /NIVARA_BOARD/ESP32 S3/RX: track 0.00 -> 21.7 mm, vias 0 -> 1
- net /NIVARA_BOARD/ESP32 S3/RELAY_OUT2: track 70.4 -> 80.3 mm
- net GND: track 152.6 -> 157.1 mm
- net /NIVARA_BOARD/ESP32 S3/PNP_OUT1: track 99.0 -> 100.9 mm
- net /NIVARA_BOARD/ESP32 S3/PNP_OUT2: track 95.0 -> 96.6 mm

Commit message: ACTUALIZACION
Routing:
- net /NIVARA_BOARD/RS_A: track 20.3 -> 16.0 mm
- net /NIVARA_BOARD/RS_B: track 15.0 -> 13.8 mm, vias 0 -> 2
Changed lines of the file:
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@@
 	(segment
 		(start 126.1234 130.111401)
-		(end 126.1234 138.188601)
+		(end 126.098 130.136801)
+		(width 0.5)
+		(layer "F.Cu")
+		(net 12)
+	)
+	(segment
+		(start 126.1234 129.197001)
+		(end 125.59 128.663601)
+		(width 0.5)
+		(layer "F.Cu")
+		(net 12)
+	)
+	(segment
+		(start 126.098 130.136801)
+		(end 126.098 138.163201)
+		(width 0.5)
+		(layer "F.Cu")
+		(net 12)
+	)
+	(segment
+		(start 122.796 127.342801)
+		(end 122.7452 127.292001)
 		(width 0.5)
 		(layer "F.Cu")
@@
 	(segment
 		(start 126.098 138.163201)
-		(end 126.098 131.406801)
-		(width 0.2)
-		(layer "F.Cu")
-		(net 12)
-	)
-	(segment
-		(start 126.1234 138.188601)
 		(end 126.1488 138.214001)
 		(width 0.5)
@@
 	)
 	(segment
-		(start 126.1488 138.214001)
-		(end 126.098 138.163201)
-		(width 0.2)
+		(start 126.1234 130.111401)
+		(end 126.1234 129.197001)
+		(width 0.5)
 		(layer "F.Cu")
 		(net 12)
 	)
 	(segment
-		(start 126.098 131.406801)
-		(end 126.1488 131.356001)
-		(width 0.2)
+		(start 123.7104 127.342801)
+		(end 122.796 127.342801)
+		(width 0.5)
 		(layer "F.Cu")
 		(net 12)
+	)
+	(via
+		(at 125.59 128.663601)
+		(size 0.6)
+		(drill 0.3)
+		(layers "F.Cu" "B.Cu")
+		(net 12)
+	)
+	(via
+		(at 123.7104 127.342801)
+		(size 0.6)
+		(drill 0.3)
+		(layers "F.Cu" "B.Cu")
+		(net 12)
+	)
+	(segment
+		(start 125.336 127.342801)
+		(end 123.7104 127.342801)
+		(width 0.5)
+		(layer "In1.Cu")
+		(net 12)
+	)
+	(segment
+		(start 125.59 127.596801)
+		(end 125.336 127.342801)
+		(width 0.5)
+		(layer "In1.Cu")
+		(net 12)
+	)
+	(segment
+		(start 125.59 128.663601)
+		(end 125.59 127.596801)
+		(width 0.5)
+		(layer "In1.Cu")
+		(net 12)
+	)
+	(segment
+		(start 123.5834 135.699401)
+		(end 121.0688 138.214001)
+		(width 0.5)
+		(layer "F.Cu")
+		(net 13)
 	)
 	(segment
@@
 	)
 	(segment
-		(start 123.5834 135.699401)
-		(end 121.0688 138.214001)
-		(width 0.5)
-		(layer "F.Cu")
-		(net 13)
-	)
-	(segment
 		(start 121.0688 138.214001)
 		(end 123.6088 135.674001)
 		(width 0.2)
 		(layer "F.Cu")
-		(net 13)
-	)
-	(segment
-		(start 123.6088 135.674001)
-		(end 123.6088 131.356001)
-		(width 0.2)
-		(layer "F.Cu")
