File: NIVARA_PCB/NIVARA/IN_DRY_Opto.kicad_sch (KiCad schematic)
At the start: 7 parts, among them U8 AT3H4A-CUH-S

Commit message: organizando componentes en la pcb
Parts:
- R16: value ? -> 1K; PART NUMBERT CRCW12061K00FKEAHP -> RC0603FR-071KL
Connections:
- net IN: now also U8.1 (A/C)
Changed lines of the file:
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@@
+	(wire
+		(pts
+			(xy 110.49 104.14) (xy 114.3 104.14)
+		)
+		(stroke
+			(width 0)
+			(type default)
+		)
+	)
 	(wire
 		(pts
@@
 			)
 		)
-		(property "Value" "?"
+		(property "Value" "1K"
 			(at 111.76 119.3799 0)
 			(effects
@@
 			)
 		)
-		(property "PART NUMBERT" "CRCW12061K00FKEAHP"
+		(property "PART NUMBERT" "RC0603FR-071KL"
 			(at 114.3 118.11 0)
 			(effects
@@
 					(unit 1)
 				)
-			)
-		)
-	)
-	(symbol
-		(lib_id "power:VCC")
-		(at 114.3 96.52 0)
-		(unit 1)
-		(exclude_from_sim no)
-		(in_bom yes)
-		(on_board yes)
-		(dnp no)
-		(fields_autoplaced yes)
-		(property "Reference" "#PWR045"
-			(at 114.3 100.33 0)
-			(effects
-				(font
-					(size 1.27 1.27)
-				)
-				(hide yes)
-			)
-		)
-		(property "Value" "VCC"
-			(at 114.3 91.44 0)
-			(effects
-				(font
-					(size 1.27 1.27)
-				)
-			)
-		)
-		(property "Footprint" ""
-			(at 114.3 96.52 0)
-			(effects
-				(font
-					(size 1.27 1.27)
-				)
-				(hide yes)
-			)
-		)
-		(property "Datasheet" ""
-			(at 114.3 96.52 0)
-			(effects
-				(font
-					(size 1.27 1.27)
-				)
-				(hide yes)
-			)
-		)
-		(property "Description" "Power symbol creates a global label with name \"VCC\""
-			(at 114.3 96.52 0)
-			(effects
-				(font
-					(size 1.27 1.27)
-				)
-				(hide yes)
-			)
-		)
-		(pin "1"
-		)
-		(instances
-			(project ""
-				(path "/6298d7d5-28da-40bf-9586-24a8e5c02b82/7ff0dada-fc46-483c-91ad-b264be8c64cf/0f260378-83c0-4366-bf66-bb63726499fd/1c6854fd-fd88-4f29-bf8b-bede240659d7"
-					(reference "#PWR045")
-					(unit 1)
-				)
-				(path "/6298d7d5-28da-40bf-9586-24a8e5c02b82/7ff0dada-fc46-483c-91ad-b264be8c64cf/0f260378-83c0-4366-bf66-bb63726499fd/7f7e2be0-af35-4d7b-9517-c789a6ac11ce"
-					(reference "#PWR046")
-					(unit 1)
-				)
