File: NIVARA_PCB/NIVARA/NIVARA_BOARD.kicad_sch (KiCad schematic)
At the start: 2 parts

Commit message: SALIDAS DE VOLTAJE Y CORRIENTE
Other:
- sheet ESP32 S3 ports: added I2C{SDA,SLCK}, NPN_OUT1, NPN_OUT2, PNP_OUT1, PNP_OUT2, RELAY_OUT1, RELAY_OUT2; removed none
- sheet OUT A 0-05V ports: added I2C{}; removed IN_1
- sheet OUT A 0-10V ports: added I2C{}; removed IN_1
- sheet OUT A 4-20mA ports: added I2C{SDA,SLCK}; removed IN_1
Changed lines of the file:
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@@
 		(color 0 0 0 0)
 	)
+	(junction
+		(at 111.76 91.44)
+		(diameter 0)
+		(color 0 0 0 0)
+	)
 	(wire
 		(pts
@@
 	(wire
 		(pts
+			(xy 106.68 133.35) (xy 116.84 133.35)
+		)
+		(stroke
+			(width 0)
+			(type default)
+		)
+	)
+	(wire
+		(pts
 			(xy 34.29 86.36) (xy 30.48 86.36)
 		)
@@
 	(wire
 		(pts
+			(xy 106.68 38.1) (xy 116.84 38.1)
+		)
+		(stroke
+			(width 0)
+			(type default)
+		)
+	)
+	(wire
+		(pts
+			(xy 106.68 31.75) (xy 116.84 31.75)
+		)
+		(stroke
+			(width 0)
+			(type default)
+		)
+	)
+	(wire
+		(pts
 			(xy 140.97 135.89) (xy 137.16 135.89)
 		)
@@
 		)
 	)
+	(bus
+		(pts
+			(xy 111.76 109.22) (xy 116.84 109.22)
+		)
+		(stroke
+			(width 0)
+			(type default)
+		)
+	)
 	(wire
 		(pts
@@
 		)
 	)
+	(bus
+		(pts
+			(xy 116.84 91.44) (xy 111.76 91.44)
+		)
+		(stroke
+			(width 0)
+			(type default)
+		)
+	)
+	(wire
+		(pts
+			(xy 140.97 125.73) (xy 137.16 125.73)
+		)
+		(stroke
+			(width 0)
+			(type default)
+		)
+	)
+	(bus
+		(pts
+			(xy 116.84 72.39) (xy 111.76 72.39)
+		)
+		(stroke
+			(width 0)
+			(type default)
+		)
+	)
+	(wire
+		(pts
+			(xy 106.68 49.53) (xy 116.84 49.53)
+		)
+		(stroke
+			(width 0)
+			(type default)
+		)
+	)
+	(wire
+		(pts
+			(xy 30.48 31.75) (xy 34.29 31.75)
+		)
+		(stroke
+			(width 0)
+			(type default)
+		)
+	)
+	(wire
+		(pts
+			(xy 140.97 133.35) (xy 137.16 133.35)
+		)
+		(stroke
+			(width 0)
+			(type default)
+		)
+	)
+	(wire
+		(pts
+			(xy 137.16 85.09) (xy 140.97 85.09)
+		)
+		(stroke
+			(width 0)
+			(type default)
+		)
+	)
+	(wire
+		(pts
+			(xy 54.61 86.36) (xy 66.04 86.36)
+		)
+		(stroke
+			(width 0)
+			(type default)
+		)
+	)
+	(wire
+		(pts
+			(xy 54.61 49.53) (xy 66.04 49.53)
+		)
+		(stroke
+			(width 0)
+			(type default)
+		)
+	)
+	(wire
+		(pts
+			(xy 30.48 138.43) (xy 34.29 138.43)
+		)
+		(stroke
+			(width 0)
+			(type default)
+		)
+	)
 	(wire
 		(pts
@@
 		)
 	)
-	(wire
-		(pts
-			(xy 140.97 125.73) (xy 137.16 125.73)
-		)
-		(stroke
-			(width 0)
-			(type default)
-		)
-	)
-	(wire
-		(pts
-			(xy 30.48 31.75) (xy 34.29 31.75)
-		)
-		(stroke
-			(width 0)
-			(type default)
-		)
-	)
-	(wire
-		(pts
-			(xy 140.97 133.35) (xy 137.16 133.35)
-		)
-		(stroke
-			(width 0)
-			(type default)
-		)
-	)
-	(wire
-		(pts
-			(xy 137.16 85.09) (xy 140.97 85.09)
-		)
-		(stroke
-			(width 0)
-			(type default)
-		)
-	)
-	(wire
-		(pts
-			(xy 54.61 86.36) (xy 66.04 86.36)
-		)
-		(stroke
-			(width 0)
-			(type default)
-		)
-	)
-	(wire
-		(pts
-			(xy 54.61 49.53) (xy 66.04 49.53)
-		)
-		(stroke
-			(width 0)
-			(type default)
-		)
-	)
-	(wire
-		(pts
-			(xy 30.48 138.43) (xy 34.29 138.43)
+	(bus
+		(pts
+			(xy 111.76 72.39) (xy 111.76 91.44)
 		)
 		(stroke
@@
 	(wire
 		(pts
+			(xy 106.68 123.19) (xy 116.84 123.19)
+		)
+		(stroke
+			(width 0)
+			(type default)
+		)
+	)
+	(wire
+		(pts
 			(xy 30.48 102.87) (xy 34.29 102.87)
 		)
@@
 		)
 	)
+	(bus
+		(pts
+			(xy 111.76 91.44) (xy 111.76 109.22)
+		)
+		(stroke
+			(width 0)
+			(type default)
+		)
+	)
 	(wire
 		(pts
@@
 		)
 	)
+	(bus
+		(pts
+			(xy 106.68 91.44) (xy 111.76 91.44)
+		)
+		(stroke
+			(width 0)
+			(type default)
+		)
+	)
 	(wire
 		(pts
@@
 		(pts
 			(xy 267.97 140.97) (xy 267.97 144.78)
+		)
+		(stroke
+			(width 0)
+			(type default)
+		)
+	)
+	(wire
+		(pts
+			(xy 106.68 55.88) (xy 116.84 55.88)
 		)
 		(stroke
@@
 			)
 		)
-		(pin "IN_1" input
-			(at 116.84 102.87 180)
-			(effects
-				(font
-					(size 1.27 1.27)
-				)
-				(justify left)
-			)
-		)
 		(pin "OUT_1" output
 			(at 137.16 102.87 0)
@@
 				)
 				(justify right)
+			)
+		)
+		(pin "I2C{SDA,SLCK}" input
+			(at 116.84 109.22 180)
+			(effects
+				(font
+					(size 1.27 1.27)
+				)
+				(justify left)
 			)
 		)
@@
 			)
 		)
-		(pin "IN_1" input
-			(at 116.84 85.09 180)
-			(effects
-				(font
-					(size 1.27 1.27)
-				)
-				(justify left)
-			)
-		)
 		(pin "OUT_1" output
 			(at 137.16 85.09 0)
@@
 				)
 				(justify right)
+			)
+		)
+		(pin "I2C{}" input
+			(at 116.84 91.44 180)
+			(effects
+				(font
+					(size 1.27 1.27)
+				)
+				(justify left)
 			)
 		)
@@
 			)
 		)
-		(pin "IN_1" input
-			(at 116.84 67.31 180)
-			(effects
-				(font
-					(size 1.27 1.27)
-				)
-				(justify left)
-			)
-		)
 		(pin "OUT_1" output
 			(at 137.16 67.31 0)
@@
 				)
 				(justify right)
+			)
+		)
+		(pin "I2C{}" input
+			(at 116.84 72.39 180)
+			(effects
+				(font
+					(size 1.27 1.27)
+				)
+				(justify left)
 			)
 		)
@@
 			)
 		)
-		(pin "A_IN4_20" input
-			(at 66.04 138.43 180)
-			(effects
-				(font
-					(size 1.27 1.27)
-				)
-				(justify left)
-			)
-		)
 		(pin "A_IN0_32" input
 			(at 66.04 120.65 180)
@@
 			(effects
 				(font
+					(size 1.27 1.27)
+				)
+				(justify left)
+			)
+		)
+		(pin "PNP_OUT1" output
+			(at 106.68 49.53 0)
+			(effects
+				(font
+					(size 1.27 1.27)
+				)
+				(justify right)
+			)
+		)
+		(pin "PNP_OUT2" output
+			(at 106.68 55.88 0)
+			(effects
+				(font
+					(size 1.27 1.27)
+				)
+				(justify right)
+			)
+		)
+		(pin "NPN_OUT2" output
+			(at 106.68 38.1 0)
+			(effects
+				(font
+					(size 1.27 1.27)
+				)
+				(justify right)
+			)
+		)
+		(pin "NPN_OUT1" output
+			(at 106.68 31.75 0)
+			(effects
+				(font
+					(size 1.27 1.27)
+				)
+				(justify right)
+			)
+		)
+		(pin "RELAY_OUT1" output
+			(at 106.68 123.19 0)
+			(effects
+				(font
+					(size 1.27 1.27)
+				)
+				(justify right)
+			)
+		)
+		(pin "RELAY_OUT2" output
+			(at 106.68 133.35 0)
+			(effects
+				(font
+					(size 1.27 1.27)
+				)
+				(justify right)
+			)
+		)
+		(pin "I2C{SDA,SLCK}" input
+			(at 106.68 91.44 0)
+			(effects
+				(font
+					(size 1.27 1.27)
+				)
+				(justify right)
+			)
+		)
+		(pin "A_IN4_20" output
+			(at 66.04 138.43 180)
+			(effects
+				(font

Commit message: Se organizaron componentes en el area de PCB
Other:
- sheet IN D renamed IN DRY
- sheet ESP32 S3 ports: added DRY_IN1, DRY_IN2; removed D_IN1, D_IN2
- sheet IN DRY: file IN_D.kicad_sch -> IN_DRY.kicad_sch
Changed lines of the file:
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@@
 			(color 0 0 0 0.0000)
 		)
-		(property "Sheetname" "IN D"
+		(property "Sheetname" "IN DRY"
 			(at 34.29 64.0584 0)
 			(effects
@@
 			)
 		)
-		(property "Sheetfile" "IN_D.kicad_sch"
+		(property "Sheetfile" "IN_DRY.kicad_sch"
 			(at 34.29 76.7846 0)
 			(effects
@@
 			)
 		)
-		(pin "D_IN2" input
-			(at 66.04 73.66 180)
-			(effects
-				(font
-					(size 1.27 1.27)
-				)
-				(justify left)
-			)
-		)
 		(pin "PNP_IN1" input
 			(at 66.04 49.53 180)
@@
 			)
 		)
-		(pin "D_IN1" input
-			(at 66.04 67.31 180)
-			(effects
-				(font
-					(size 1.27 1.27)
-				)
-				(justify left)
-			)
-		)
 		(pin "NPN_IN1" input
 			(at 66.04 31.75 180)
@@
 			)
 		)
-		(pin "A_IN4_20" output
+		(pin "A_IN4_20" input
 			(at 66.04 138.43 180)
 			(effects
 				(font
+					(size 1.27 1.27)
+				)
+				(justify left)
+			)
+		)
+		(pin "DRY_IN2" input
+			(at 66.04 73.66 180)
+			(effects
+				(font
+					(size 1.27 1.27)
+				)
+				(justify left)
+			)
+		)
+		(pin "DRY_IN1" input
+			(at 66.04 67.31 180)
+			(effects
+				(font

Commit message: arreglo del desastre que tenia con las salidas PNP
Other:
- sheet OUT A 0-05V ports: added I2C{SDA,SLCK}; removed I2C{}
- sheet OUT A 0-10V ports: added I2C{SDA,SLCK}; removed I2C{}
Changed lines of the file:
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@@
 	(bus
 		(pts
-			(xy 116.84 91.44) (xy 111.76 91.44)
+			(xy 111.76 91.44) (xy 116.84 91.44)
 		)
 		(stroke
@@
 		)
 	)
+	(bus
+		(pts
+			(xy 111.76 72.39) (xy 111.76 91.44)
+		)
+		(stroke
+			(width 0)
+			(type default)
+		)
+	)
 	(wire
 		(pts
@@
 		(pts
 			(xy 54.61 138.43) (xy 66.04 138.43)
-		)
-		(stroke
-			(width 0)
-			(type default)
-		)
-	)
-	(bus
-		(pts
-			(xy 111.76 72.39) (xy 111.76 91.44)
 		)
 		(stroke
@@
 			)
 		)
-		(pin "I2C{}" input
+		(pin "I2C{SDA,SLCK}" input
 			(at 116.84 91.44 180)
 			(effects
@@
 			)
 		)
-		(pin "I2C{}" input
+		(pin "I2C{SDA,SLCK}" input
 			(at 116.84 72.39 180)
 			(effects
