File: NIVARA_PCB/NIVARA/OUTA0-10V.kicad_sch (KiCad schematic)
At the start: 0 parts

Commit message: avance
Parts:
- added U10: GP8201S-TC50-EW, easyeda2kicad:ESOP-8_L4.9-W3.9-P1.27-LS6.0-BL-EP, symbol easyeda2kicad:GP8201S-TC50-EW
Connections:
- net OUT_1: now also U10.6 (VOUT)
- new net GND: U10.5 (GND)
- new net SCLK: U10.1 (SCLK)
- new net SDA: U10.2 (SDA)
- new net VCC: U10.4 (VCC)
- no-connect marks 0 -> 1

Commit message: SALIDAS DE VOLTAJE Y CORRIENTE
Parts:
- added C19: 1uF, PCM_Capacitor_SMD_AKL:C_0603_1608Metric, symbol PCM_Capacitor_AKL:C_0603
- added C20: 100nF, PCM_Capacitor_SMD_AKL:C_0603_1608Metric, symbol PCM_Capacitor_AKL:C_0603
- added D6: SM6T12A, Diode_SMD:D_SMB, symbol Diode:SM6T12A
- added R14: 0R, PCM_Resistor_SMD_AKL:R_0603_1608Metric, symbol PCM_Resistor_AKL:R_0603
Connections:
- net GND: now also U10.9 (EP), C19.1, C20.1, D6.2 (A2)
- net OUT_1: now also C20.2, D6.1 (A1)
- net at U10.7 (SEL): now also R14.2
- net at U10.8 (V5V): now also C19.2, R14.1
- net SCLK renamed I2C.SLCK
- net SDA renamed I2C.SDA

Commit message: ACTUALIZACION
Parts:
- C20: PART NUMBERT (none) -> CC0603KRX7R9BB104
Changed lines of the file:
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@@
 			)
 		)
-		(property "PART NUMBERT" ""
+		(property "PART NUMBERT" "CC0603KRX7R9BB104"
 			(at 78.74 54.61 0)
 			(effects
@@
 					(size 1.27 1.27)
 				)
+				(hide yes)
 			)
 		)

Commit message: arreglo del desastre que tenia con las salidas PNP
Parts:
- removed D6: SM6T12A, Diode_SMD:D_SMB, symbol Diode:SM6T12A
- added D6: SMF11A, PCM_Diode_SMD_AKL:D_SOD-123F, symbol PCM_Diode_TVS_AKL:SMF11A
Connections:
- net GND: now also D6.2 (A)
- net OUT_1: now also D6.1 (K)
- no-connect marks 1 -> 0
Changed lines of the file:
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@@
 		(color 0 0 0 0)
-	)
-	(no_connect
-		(at 33.02 50.8)
-	)
-	(bus_entry
-		(at 21.59 45.72)
-		(size 2.54 2.54)
-		(stroke
-			(width 0)
-			(type default)
-		)
 	)
 	(bus_entry
@@
 		)
 	)
+	(bus_entry
+		(at 21.59 44.45)
+		(size 2.54 2.54)
+		(stroke
+			(width 0)
+			(type default)
+		)
+	)
 	(wire
 		(pts
@@
 		)
 	)
+	(wire
+		(pts
+			(xy 24.13 45.72) (xy 33.02 45.72)
+		)
+		(stroke
+			(width 0)
+			(type default)
+		)
+	)
+	(wire
+		(pts
+			(xy 24.13 48.26) (xy 33.02 48.26)
+		)
+		(stroke
+			(width 0)
+			(type default)
+		)
+	)
+	(wire
+		(pts
+			(xy 87.63 50.8) (xy 107.95 50.8)
+		)
+		(stroke
+			(width 0)
+			(type default)
+		)
+	)
+	(wire
+		(pts
+			(xy 33.02 55.88) (xy 33.02 53.34)
+		)
+		(stroke
+			(width 0)
+			(type default)
+		)
+	)
 	(bus
 		(pts
+			(xy 21.59 43.18) (xy 21.59 44.45)
+		)
+		(stroke
+			(width 0)
+			(type default)
+		)
+	)
+	(wire
+		(pts
+			(xy 55.88 31.75) (xy 55.88 43.18)
+		)
+		(stroke
+			(width 0)
+			(type default)
+		)
+	)
+	(bus
+		(pts
 			(xy 21.59 40.64) (xy 21.59 43.18)
 		)
@@
 	(wire
 		(pts
-			(xy 87.63 50.8) (xy 107.95 50.8)
-		)
-		(stroke
-			(width 0)
-			(type default)
-		)
-	)
-	(wire
-		(pts
-			(xy 33.02 55.88) (xy 33.02 53.34)
-		)
-		(stroke
-			(width 0)
-			(type default)
-		)
-	)
-	(wire
-		(pts
-			(xy 55.88 31.75) (xy 55.88 43.18)
+			(xy 55.88 55.88) (xy 55.88 53.34)
+		)
+		(stroke
+			(width 0)
+			(type default)
+		)
+	)
+	(wire
+		(pts
+			(xy 78.74 50.8) (xy 87.63 50.8)
+		)
+		(stroke
+			(width 0)
+			(type default)
+		)
+	)
+	(wire
+		(pts
+			(xy 24.13 46.99) (xy 24.13 48.26)
+		)
+		(stroke
+			(width 0)
+			(type default)
+		)
+	)
+	(wire
+		(pts
+			(xy 55.88 45.72) (xy 58.42 45.72)
+		)
+		(stroke
+			(width 0)
+			(type default)
+		)
+	)
+	(wire
+		(pts
+			(xy 58.42 40.64) (xy 60.96 40.64)
+		)
+		(stroke
+			(width 0)
+			(type default)
+		)
+	)
+	(wire
+		(pts
+			(xy 58.42 45.72) (xy 58.42 40.64)
 		)
 		(stroke
@@
 	(bus
 		(pts
-			(xy 21.59 43.18) (xy 21.59 45.72)
-		)
-		(stroke
-			(width 0)
-			(type default)
-		)
-	)
-	(wire
-		(pts
-			(xy 55.88 55.88) (xy 55.88 53.34)
-		)
-		(stroke
-			(width 0)
-			(type default)
-		)
-	)
-	(wire
-		(pts
-			(xy 78.74 50.8) (xy 87.63 50.8)
-		)
-		(stroke
-			(width 0)
-			(type default)
-		)
-	)
-	(wire
-		(pts
-			(xy 55.88 45.72) (xy 58.42 45.72)
-		)
-		(stroke
-			(width 0)
-			(type default)
-		)
-	)
-	(wire
-		(pts
-			(xy 24.13 48.26) (xy 33.02 48.26)
-		)
-		(stroke
-			(width 0)
-			(type default)
-		)
-	)
-	(wire
-		(pts
-			(xy 58.42 40.64) (xy 60.96 40.64)
-		)
-		(stroke
-			(width 0)
-			(type default)
-		)
-	)
-	(wire
-		(pts
-			(xy 58.42 45.72) (xy 58.42 40.64)
-		)
-		(stroke
-			(width 0)
-			(type default)
-		)
-	)
-	(wire
-		(pts
-			(xy 24.13 45.72) (xy 33.02 45.72)
+			(xy 21.59 44.45) (xy 21.59 45.72)
 		)
 		(stroke
@@
 		)
 	)
-	(label "I2C.SLCK"
-		(at 33.02 45.72 180)
+	(label "I2C.SDA"
+		(at 33.02 48.26 0)
 		(effects
 			(font
 				(size 1.27 1.27)
 			)
-			(justify right bottom)
-		)
-	)
-	(label "I2C.SDA"
-		(at 33.02 48.26 180)
+			(justify left bottom)
+		)
+	)
+	(label "I2C.SLCK"
+		(at 33.02 45.72 0)
 		(effects
 			(font
 				(size 1.27 1.27)
 			)
-			(justify right bottom)
+			(justify left bottom)
 		)
 	)
@@
 		)
 	)
-	(hierarchical_label "I2C{}"
+	(hierarchical_label "I2C{SDA,SLCK}"
 		(shape input)
 		(at 21.59 40.64 90)
@@
 			)
 			(justify left)
+		)
+	)
+	(symbol
+		(lib_id "PCM_Diode_TVS_AKL:SMF11A")
+		(at 87.63 54.61 90)
+		(unit 1)
+		(exclude_from_sim no)
+		(in_bom yes)
+		(on_board yes)
+		(dnp no)
+		(fields_autoplaced yes)
+		(property "Reference" "D6"
+			(at 90.17 53.3399 90)
+			(effects
+				(font
+					(size 1.27 1.27)
+				)
+				(justify right)
+			)
+		)
+		(property "Value" "SMF11A"
+			(at 90.17 55.8799 90)
+			(effects
+				(font
+					(size 1.27 1.27)
+				)
+				(justify right)
+			)
+		)
+		(property "Footprint" "PCM_Diode_SMD_AKL:D_SOD-123F"
+			(at 87.63 54.61 0)
+			(effects
+				(font
+					(size 1.27 1.27)
+				)
+				(hide yes)
+			)
+		)
+		(property "Datasheet" "https://www.tme.eu/Document/95faf1e5e821ed1b438500c66c7b0bd9/smf50a.pdf"
+			(at 87.63 54.61 0)
+			(effects
+				(font
+					(size 1.27 1.27)
+				)
+				(hide yes)
+			)
+		)
+		(property "Description" "SOD-123F Unidirectional TVS diode, 11V, 200W, Alternate KiCAD Library"
+			(at 87.63 54.61 0)
+			(effects
+				(font
+					(size 1.27 1.27)
+				)
+				(hide yes)
+			)
+		)
+		(pin "2"
+		)
+		(pin "1"
+		)
+		(instances
+			(project ""
+				(path "/6298d7d5-28da-40bf-9586-24a8e5c02b82/7ff0dada-fc46-483c-91ad-b264be8c64cf/27fcba6f-4116-4b57-87c7-0cd3789c6248"
+					(reference "D6")
+					(unit 1)
+				)
+			)
 		)
 	)
@@
 					(unit 1)
 				)
-			)
-		)
-	)
-	(symbol
-		(lib_id "Diode:SM6T12A")
-		(at 87.63 54.61 270)
-		(unit 1)
-		(exclude_from_sim no)
-		(in_bom yes)
-		(on_board yes)
-		(dnp no)
-		(fields_autoplaced yes)
-		(property "Reference" "D6"
-			(at 90.17 53.3399 90)
-			(effects
-				(font
-					(size 1.27 1.27)
-				)
-				(justify left)
-			)
-		)
-		(property "Value" "SM6T12A"
-			(at 90.17 55.8799 90)
-			(effects
-				(font
-					(size 1.27 1.27)
-				)
-				(justify left)
-			)
-		)
-		(property "Footprint" "Diode_SMD:D_SMB"
-			(at 82.55 54.61 0)
-			(effects
-				(font
-					(size 1.27 1.27)
-				)
-				(hide yes)
-			)
-		)
-		(property "Datasheet" "https://www.st.com/resource/en/datasheet/sm6t.pdf"
-			(at 87.63 53.34 0)
-			(effects
-				(font
-					(size 1.27 1.27)
-				)
-				(hide yes)
-			)
-		)
-		(property "Description" "600W unidirectional Transil Transient Voltage Suppressor, 12Vrwm, DO-214AA"
-			(at 87.63 54.61 0)
-			(effects
-				(font
-					(size 1.27 1.27)
-				)
-				(hide yes)
-			)
-		)
-		(pin "2"
-		)
-		(pin "1"
-		)
-		(instances
-			(project ""
-				(path "/6298d7d5-28da-40bf-9586-24a8e5c02b82/7ff0dada-fc46-483c-91ad-b264be8c64cf/27fcba6f-4116-4b57-87c7-0cd3789c6248"
-					(reference "D6")
-					(unit 1)
-				)
