File: NIVARA_PCB/NIVARA/OUTA4-20mA.kicad_sch (KiCad schematic)
At the start: 0 parts

Commit message: avance
Parts:
- added U9: GP8303-TC50-EW, easyeda2kicad:ESOP-10_L4.9-W3.9-P1.00-LS6.1-BL-EP, symbol easyeda2kicad:GP8303-TC50-EW
Connections:
- net OUT_1: now also U9.8 (IOUT)
- new net A0: U9.3 (A0)
- new net A1: U9.4 (A1)
- new net A2: U9.9 (A2)
- new net SDA: U9.2 (SDA)
- new net SLCK: U9.1 (SLCK)
- new net VCC: U9.5 (VCC)

Commit message: SALIDAS DE VOLTAJE Y CORRIENTE
Parts:
- added C16: 220uF, PCM_Capacitor_SMD_AKL:C_0603_1608Metric, symbol PCM_Capacitor_AKL:C_0603
- added C17, C9: 1uF, PCM_Capacitor_SMD_AKL:C_0603_1608Metric, symbol PCM_Capacitor_AKL:C_0603
- added C18: 100nF, PCM_Capacitor_SMD_AKL:C_0603_1608Metric, symbol PCM_Capacitor_AKL:C_0603
- added D4: 1N4007, Diode_SMD:D_SOD-123F, symbol PCM_Diode_AKL:1N4007
- added D5: SM6T24A, Diode_SMD:D_SMB, symbol Diode:SM6T24A
- added JP2: A0, Jumper:SolderJumper-2_P1.3mm_Open_RoundedPad1.0x1.5mm, symbol Jumper:SolderJumper_2_Open
- added JP3: A1, Jumper:SolderJumper-2_P1.3mm_Open_RoundedPad1.0x1.5mm, symbol Jumper:SolderJumper_2_Open
- added JP4: A2, Jumper:SolderJumper-2_P1.3mm_Open_RoundedPad1.0x1.5mm, symbol Jumper:SolderJumper_2_Open
- added Q3: BRCS4435SC, easyeda2kicad:SOP-8_L5.0-W4.0-P1.27-LS6.0-BL, symbol easyeda2kicad:BRCS4435SC
- added R10, R8, R9: 1K, PCM_Resistor_SMD_AKL:R_1206_3216Metric_Pad1.30x1.75mm_HandSolder, symbol PCM_Resistor_AKL:R_0603
- added R11: 2.5K, PCM_Resistor_SMD_AKL:R_0603_1608Metric, symbol PCM_Resistor_AKL:R_0603
- added R12: 100K, PCM_Resistor_SMD_AKL:R_0603_1608Metric, symbol PCM_Resistor_AKL:R_0603
- added R13: 15R, PCM_Resistor_SMD_AKL:R_1206_3216Metric, symbol PCM_Resistor_AKL:R_1206
- added U12: ZMM12V_C5345999, easyeda2kicad:LL-34_L3.5-W1.5-RD-2, symbol easyeda2kicad:ZMM12V_C5345999
Connections:
- net A0: now also JP2.2 (B), R8.2
- net A1: now also JP3.2 (B), R9.2
- net A2: now also JP4.2 (B), R10.2
- net OUT_1: now also D4.1 (K); no longer U9.8 (IOUT)
- net VCC: now also U12.1 (K)
- net at U9.10 (V5V): now also C9.2
- net GND: now reaches U9.11 (EP)
- net GND: now also U9.6 (GND), C16.2, C17.2, C18.1, C9.1, D5.2 (A2), R10.1, R11.2, R12.2, R8.1, R9.1
- net at U9.7 (SET): now also C16.1, R11.1
- net SDA renamed I2C.SDA
- net SLCK renamed I2C.SLCK
- new net: Q3.1 (S), Q3.2 (S), Q3.3 (S), U9.8 (IOUT)
- new net: C17.1, Q3.4 (G), R12.1, U12.2 (A)
- new net: C18.2, D5.1 (A1), Q3.5 (D), Q3.6 (D), Q3.7 (D), Q3.8 (D), R13.1
- new net: D4.2 (A), R13.2
- new net +3V3: JP2.1 (A), JP3.1 (A), JP4.1 (A)

Commit message: ACTUALIZACION
Parts:
- C18: PART NUMBERT (none) -> CC0603KRX7R9BB104
Changed lines of the file:
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@@
 			)
 		)
-		(property "PART NUMBERT" ""
+		(property "PART NUMBERT" "CC0603KRX7R9BB104"
 			(at 111.76 46.99 0)
 			(effects

Commit message: Se organizaron componentes en el area de PCB
Parts:
- R10, R8, R9: footprint PCM_Resistor_SMD_AKL:R_1206_3216Metric_Pad1.30x1.75mm_HandSolder -> PCM_Resistor_SMD_AKL:R_0603_1608Metric; PART NUMBERT CRCW12061K00FKEAHP -> RC0603FR-071KL
Changed lines of the file:
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@@
 			)
 		)
-		(property "Footprint" "PCM_Resistor_SMD_AKL:R_1206_3216Metric_Pad1.30x1.75mm_HandSolder"
+		(property "Footprint" "PCM_Resistor_SMD_AKL:R_0603_1608Metric"
 			(at 10.16 77.47 0)
 			(effects
@@
 			)
 		)
-		(property "PART NUMBERT" "CRCW12061K00FKEAHP"
+		(property "PART NUMBERT" "RC0603FR-071KL"
 			(at 21.59 77.47 0)
 			(effects
@@
 			)
 		)
-		(property "Footprint" "PCM_Resistor_SMD_AKL:R_1206_3216Metric_Pad1.30x1.75mm_HandSolder"
+		(property "Footprint" "PCM_Resistor_SMD_AKL:R_0603_1608Metric"
 			(at 31.75 77.47 0)
 			(effects
@@
 			)
 		)
-		(property "PART NUMBERT" "CRCW12061K00FKEAHP"
+		(property "PART NUMBERT" "RC0603FR-071KL"
 			(at 43.18 77.47 0)
 			(effects
@@
 			)
 		)
-		(property "Footprint" "PCM_Resistor_SMD_AKL:R_1206_3216Metric_Pad1.30x1.75mm_HandSolder"
+		(property "Footprint" "PCM_Resistor_SMD_AKL:R_0603_1608Metric"
 			(at 20.32 77.47 0)
 			(effects
@@
 			)
 		)
-		(property "PART NUMBERT" "CRCW12061K00FKEAHP"
+		(property "PART NUMBERT" "RC0603FR-071KL"
 			(at 31.75 77.47 0)
 			(effects

Commit message: arreglo del desastre que tenia con las salidas PNP
Parts:
- removed D5: SM6T24A, Diode_SMD:D_SMB, symbol Diode:SM6T24A
- removed Q3: BRCS4435SC, easyeda2kicad:SOP-8_L5.0-W4.0-P1.27-LS6.0-BL, symbol easyeda2kicad:BRCS4435SC
- added D7: SMF24A, Diode_SMD:D_SMF, symbol Diode:SMF24A
- added Q1: DMP3056L, PCM_Package_TO_SOT_SMD_AKL:SOT-23, symbol PCM_Transistor_MOSFET_AKL:DMP3056L
Connections:
- net GND: now also D7.2 (A2)
- net at U9.8 (IOUT): now also Q1.2 (S)
- net at C17.1, R12.1, U12.2 (A): now also Q1.1 (G)
- net at C18.2, R13.1: now also D7.1 (A1), Q1.3 (D)
Other:
- moved on the sheet: C17, C18, D4, R12, R13, U12
