File: NIVARA_PCB/NIVARA/O_NPN.kicad_sch (KiCad schematic)
At the start: 3 parts, among them Q5 NCV8402xST

Commit message: arreglo del desastre que tenia con las salidas PNP
Parts:
- removed Q5: NCV8402xST, Package_TO_SOT_SMD:SOT-223, symbol Driver_FET:NCV8402xST
- added U14: ZXMS6004FFQTA, easyeda2kicad:SOT-23F_L2.9-W1.8-P0.95-LS2.4-BR, symbol CUSTOM:ZXMS6004FFQTA
Connections:
- net GND: now also U14.2 (S)
- net OUT: now also U14.3 (D)
- net at R31.1, R36.1: now also U14.1 (IN)
Changed lines of the file:
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@@
 	(wire
 		(pts
-			(xy 76.2 52.07) (xy 81.28 52.07)
+			(xy 76.2 52.07) (xy 87.63 52.07)
 		)
 		(stroke
@@
 	(wire
 		(pts
-			(xy 101.6 35.56) (xy 101.6 41.91)
+			(xy 101.6 35.56) (xy 101.6 45.72)
 		)
 		(stroke
@@
 	(wire
 		(pts
-			(xy 101.6 67.31) (xy 101.6 62.23)
+			(xy 101.6 58.42) (xy 101.6 67.31)
 		)
 		(stroke
@@
 	)
 	(symbol
-		(lib_id "Driver_FET:NCV8402xST")
-		(at 93.98 52.07 0)
+		(lib_id "CUSTOM:ZXMS6004FFQTA")
+		(at 96.52 52.07 0)
 		(unit 1)
 		(exclude_from_sim no)
@@
 		(dnp no)
 		(fields_autoplaced yes)
-		(property "Reference" "Q5"
-			(at 105.41 50.7999 0)
+		(property "Reference" "U14"
+			(at 104.14 50.7999 0)
 			(effects
 				(font
@@
 			)
 		)
-		(property "Value" "NCV8402xST"
-			(at 105.41 53.3399 0)
+		(property "Value" "ZXMS6004FFQTA"
+			(at 104.14 53.3399 0)
 			(effects
 				(font
@@
 			)
 		)
-		(property "Footprint" "Package_TO_SOT_SMD:SOT-223"
-			(at 93.98 59.182 0)
-			(effects
-				(font
-					(size 1.27 1.27)
-				)
-				(hide yes)
-			)
-		)
-		(property "Datasheet" "https://www.onsemi.com/pub/Collateral/NCV8402-D.PDF"
-			(at 101.6 52.07 0)
-			(effects
-				(font
-					(size 1.27 1.27)
-				)
-				(hide yes)
-			)
-		)
-		(property "Description" "Self-Protected Low Side Driver with Temperature and Current Limit, SOT−223"
-			(at 93.98 52.07 0)
+		(property "Footprint" "easyeda2kicad:SOT-23F_L2.9-W1.8-P0.95-LS2.4-BR"
+			(at 96.52 52.07 0)
+			(effects
+				(font
+					(size 1.27 1.27)
+				)
+				(hide yes)
+			)
+		)
+		(property "Datasheet" "https://www.lcsc.com/datasheet/C508259.pdf"
+			(at 96.52 52.07 0)
+			(effects
+				(font
+					(size 1.27 1.27)
+				)
+				(hide yes)
+			)
+		)
+		(property "Description" "The DIODES™ ZXMS6004FFQ is a self-protected low side IntelliFET™ MOSFET with logic level input. It integrates overtemperature, overcurrent, overvoltage (active clamp) and ESD protected logic level functionality. The ZXMS6004FFQ is ideal as a general purpose switch driven from 3.3V or 5V microcontrollers in harsh environments where standard MOSFETs are not rugged enough."
+			(at 96.52 52.07 0)
 			(effects
 				(font
@@
 		(pin "3"
 		)
+		(pin "2"
+		)
 		(pin "1"
-		)
-		(pin "2"
-		)
-		(pin "4"
 		)
 		(instances
 			(project ""
 				(path "/6298d7d5-28da-40bf-9586-24a8e5c02b82/7ff0dada-fc46-483c-91ad-b264be8c64cf/e83b750d-d99e-4d1f-827c-e43e7f4ff994/62e5c501-aff0-4998-8240-061b2af6ecfc"
-					(reference "Q8")
+					(reference "U15")
 					(unit 1)
 				)
 				(path "/6298d7d5-28da-40bf-9586-24a8e5c02b82/7ff0dada-fc46-483c-91ad-b264be8c64cf/e83b750d-d99e-4d1f-827c-e43e7f4ff994/810b091e-4bcf-48f8-b7f3-b9f1b9e09f44"
-					(reference "Q5")
-					(unit 1)
-				)
+					(reference "U14")
+					(unit 1)
+				)
