File: NIVARA_PCB/NIVARA/_autosave-NIVARA.kicad_pcb (KiCad board)
At the start: 4 copper layers, 101.2 x 82 mm, 200 parts, among them IC1 ITS5215, J1 Power, J10 I_ANALOG, J11 RS485, J12 O_ANALOG, J3 I_NPN, J4 I_PNP, J5 RELAY_1, J6 RELAY_2, J7 O_NPN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

Commit message: ruteo de salidas
Connections:
- U11 pad 10: /NIVARA_BOARD/ESP32 S3/NPN_OUT2 -> /NIVARA_BOARD/ESP32 S3/NPN_OUT1
- U11 pad 11: /NIVARA_BOARD/ESP32 S3/NPN_OUT1 -> /NIVARA_BOARD/ESP32 S3/NPN_OUT2
Routing:
- net /NIVARA_BOARD/ESP32 S3/NPN_OUT2: track 0.00 -> 113.9 mm, vias 0 -> 2
- net /NIVARA_BOARD/ESP32 S3/NPN_OUT1: track 0.00 -> 111.3 mm, vias 0 -> 2
- net /NIVARA_BOARD/ESP32 S3/RELAY_OUT2: track 70.4 -> 80.3 mm
- net GND: track 152.6 -> 157.1 mm
- net /NIVARA_BOARD/ESP32 S3/PNP_OUT1: track 99.0 -> 100.9 mm
- net /NIVARA_BOARD/ESP32 S3/PNP_OUT2: track 95.0 -> 96.6 mm
