File: NIVARA_PCB/NIVARA/_autosave-ESP32_S3.kicad_sch (KiCad schematic)
At the start: 8 parts, among them U11 ESP32-S3-WROOM-1

Commit message: RUTEO ENTRADAS
Connections:
- net DRY_IN1: now also U11.21 (GPIO13/TOUCH13/ADC2_CH2/FSPIQ/FSPIIO7/SUBSPIQ)
- net DRY_IN2: now also U11.20 (GPIO12/TOUCH12/ADC2_CH1/FSPICLK/FSPIIO6/SUBSPICLK)
Changed lines of the file:
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@@
+	(wire
+		(pts
+			(xy 163.83 92.71) (xy 158.75 92.71)
+		)
+		(stroke
+			(width 0)
+			(type default)
+		)
+	)
 	(wire
 		(pts
@@
 		(pts
 			(xy 161.29 105.41) (xy 158.75 105.41)
+		)
+		(stroke
+			(width 0)
+			(type default)
+		)
+	)
+	(wire
+		(pts
+			(xy 163.83 95.25) (xy 158.75 95.25)
 		)
 		(stroke
@@
 		)
 	)
-	(hierarchical_label "DRY_IN2"
-		(shape input)
-		(at 27.94 87.63 180)
-		(effects
-			(font
-				(size 1.27 1.27)
-			)
-			(justify right)
-		)
-	)
 	(hierarchical_label "RX"
 		(shape bidirectional)
@@
 		)
 	)
+	(hierarchical_label "DRY_IN1"
+		(shape input)
+		(at 163.83 95.25 0)
+		(effects
+			(font
+				(size 1.27 1.27)
+			)
+			(justify left)
+		)
+	)
 	(hierarchical_label "NPN_OUT2"
 		(shape output)
@@
 		(shape input)
 		(at 161.29 67.31 0)
+		(effects
+			(font
+				(size 1.27 1.27)
+			)
+			(justify left)
+		)
+	)
+	(hierarchical_label "DRY_IN2"
+		(shape input)
+		(at 163.83 92.71 0)
 		(effects
 			(font
@@
 		)
 	)
-	(hierarchical_label "DRY_IN1"
-		(shape input)
-		(at 27.94 81.28 180)
-		(effects
-			(font
-				(size 1.27 1.27)
-			)
-			(justify right)
-		)
-	)
